Commit message: trial

File: urdf_to_mjcf/tests/piper_description.urdf (robot description, URDF)
Before this commit: robot piper, 10 links, 9 joints
Links:
- removed link base_link
- removed link gripper_base
- removed link link1
- removed link link2
- removed link link3
- removed link link4
- removed link link5
- removed link link6
- removed link link7
- removed link link8
- added link left_base_link, mass 0.018515312401126; collision mesh filename=package://visualization/urdf/left_hand_v1_meshes/base_link.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; visual mesh filename=package://visualization/urdf/left_hand_v1_meshes/base_link.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
- added link left_frame_link, mass 0.046182728238364; collision mesh filename=package://visualization/urdf/left_hand_v1_meshes/frame_link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; visual mesh filename=package://visualization/urdf/left_hand_v1_meshes/frame_link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
- added link left_index_distal_link, mass 0.00137698971613404; collision mesh filename=package://visualization/urdf/left_hand_v1_meshes/index_dist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; visual mesh filename=package://visualization/urdf/left_hand_v1_meshes/index_dist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
- added link left_index_f_link, mass 0.000272618505177845; collision mesh filename=package://visualization/urdf/left_hand_v1_meshes/index_f_li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; visual mesh filename=package://visualization/urdf/left_hand_v1_meshes/index_f_li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
- added link left_index_middle_link, mass 0.0022951205465851; collision mesh filename=package://visualization/urdf/left_hand_v1_meshes/index_midd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; visual mesh filename=package://visualization/urdf/left_hand_v1_meshes/index_midd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
- added link left_index_prismatic1_link, mass 0.000394369846861351; collision mesh filename=package://visualization/urdf/left_hand_v1_meshes/index_pris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; visual mesh filename=package://visualization/urdf/left_hand_v1_meshes/index_pris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
- added link left_index_prismatic2_link, mass 0.000394369846861351; collision mesh filename=package://visualization/urdf/left_hand_v1_meshes/index_pris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; visual mesh filename=package://visualization/urdf/left_hand_v1_meshes/index_pris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
- added link left_index_proximal_link, mass 0.00599684399920735; collision mesh filename=package://visualization/urdf/left_hand_v1_meshes/index_prox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; visual mesh filename=package://visualization/urdf/left_hand_v1_meshes/index_prox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
- added link left_index_tip_link, mass 0.00170572301090788; collision mesh filename=package://visualization/urdf/left_hand_v1_meshes/index_tip_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; visual mesh filename=package://visualization/urdf/left_hand_v1_meshes/index_tip_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
- added link left_middle_distal_link, mass 0.00137698810312193; collision mesh filename=package://visualization/urdf/left_hand_v1_meshes/middle_dis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; visual mesh filename=package://visualization/urdf/left_hand_v1_meshes/middle_dis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
- added link left_middle_f_link, mass 0.000272618505177845; collision mesh filename=package://visualization/urdf/left_hand_v1_meshes/middle_f_l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; visual mesh filename=package://visualization/urdf/left_hand_v1_meshes/middle_f_l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
- added link left_middle_middle_link, mass 0.00229512127249161; collision mesh filename=package://visualization/urdf/left_hand_v1_meshes/middle_mid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; visual mesh filename=package://visualization/urdf/left_hand_v1_meshes/middle_mid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
- added link left_middle_prismatic1_link, mass 0.000394369846861353; collision mesh filename=package://visualization/urdf/left_hand_v1_meshes/middle_pri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; visual mesh filename=package://visualization/urdf/left_hand_v1_meshes/middle_pri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
- added link left_middle_prismatic2_link, mass 0.000394369846861354; collision mesh filename=package://visualization/urdf/left_hand_v1_meshes/middle_pri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; visual mesh filename=package://visualization/urdf/left_hand_v1_meshes/middle_pri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
- added link left_middle_proximal_link, mass 0.00599684490093027; collision mesh filename=package://visualization/urdf/left_hand_v1_meshes/middle_pro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; visual mesh filename=package://visualization/urdf/left_hand_v1_meshes/middle_pro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
- added link left_middle_tip_link, mass 0.00170572337119633; collision mesh filename=package://visualization/urdf/left_hand_v1_meshes/middle_tip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; visual mesh filename=package://visualization/urdf/left_hand_v1_meshes/middle_tip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
- added link left_pinky_distal_link, mass 0.00137698956250512; collision mesh filename=package://visualization/urdf/left_hand_v1_meshes/pinky_dist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; visual mesh filename=package://visualization/urdf/left_hand_v1_meshes/pinky_dist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
- added link left_pinky_f_link, mass 0.000272618505177846; collision mesh filename=package://visualization/urdf/left_hand_v1_meshes/pinky_f_li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; visual mesh filename=package://visualization/urdf/left_hand_v1_meshes/pinky_f_li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
- added link left_pinky_middle_link, mass 0.00229511880358933; collision mesh filename=package://visualization/urdf/left_hand_v1_meshes/pinky_midd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; visual mesh filename=package://visualization/urdf/left_hand_v1_meshes/pinky_midd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
- added link left_pinky_prismatic1_link, mass 0.000394369846861354; collision mesh filename=package://visualization/urdf/left_hand_v1_meshes/pinky_pris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; visual mesh filename=package://visualization/urdf/left_hand_v1_meshes/pinky_pris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
- added link left_pinky_prismatic2_link, mass 0.000394369846861356; collision mesh filename=package://visualization/urdf/left_hand_v1_meshes/pinky_pris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; visual mesh filename=package://visualization/urdf/left_hand_v1_meshes/pinky_pris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
- added link left_pinky_proximal_link, mass 0.00599683372090147; collision mesh filename=package://visualization/urdf/left_hand_v1_meshes/pinky_prox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; visual mesh filename=package://visualization/urdf/left_hand_v1_meshes/pinky_prox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
- added link left_pinky_tip_link, mass 0.00170572327227634; collision mesh filename=package://visualization/urdf/left_hand_v1_meshes/pinky_tip_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; visual mesh filename=package://visualization/urdf/left_hand_v1_meshes/pinky_tip_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
- added link left_ring_distal_link, mass 0.00137698874426085; collision mesh filename=package://visualization/urdf/left_hand_v1_meshes/ring_dista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; visual mesh filename=package://visualization/urdf/left_hand_v1_meshes/ring_dista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
- added link left_ring_f_link, mass 0.000272618505177846; collision mesh filename=package://visualization/urdf/left_hand_v1_meshes/ring_f_lin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; visual mesh filename=package://visualization/urdf/left_hand_v1_meshes/ring_f_lin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
- added link left_ring_middle_link, mass 0.00229512027057487; collision mesh filename=package://visualization/urdf/left_hand_v1_meshes/ring_middl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; visual mesh filename=package://visualization/urdf/left_hand_v1_meshes/ring_middl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
- added link left_ring_prismatic1_link, mass 0.000394369846861354; collision mesh filename=package://visualization/urdf/left_hand_v1_meshes/ring_prism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; visual mesh filename=package://visualization/urdf/left_hand_v1_meshes/ring_prism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
- added link left_ring_prismatic2_link, mass 0.000394369846861355; collision mesh filename=package://visualization/urdf/left_hand_v1_meshes/ring_prism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; visual mesh filename=package://visualization/urdf/left_hand_v1_meshes/ring_prism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
- added link left_ring_proximal_link, mass 0.00599684572639037; collision mesh filename=package://visualization/urdf/left_hand_v1_meshes/ring_proxi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; visual mesh filename=package://visualization/urdf/left_hand_v1_meshes/ring_proxi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
- added link left_ring_tip_link, mass 0.00170572318511849; collision mesh filename=package://visualization/urdf/left_hand_v1_meshes/ring_tip_l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; visual mesh filename=package://visualization/urdf/left_hand_v1_meshes/ring_tip_l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
- added link left_t_Link, mass 0.00253406620111725; collision mesh filename=package://visualization/urdf/left_hand_v1_meshes/t_Link.STL; visual mesh filename=package://visualization/urdf/left_hand_v1_meshes/t_Link.STL
- added link left_thumb_distal_link, mass 0.00364556544568981; collision mesh filename=package://visualization/urdf/left_hand_v1_meshes/thumb_dist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; visual mesh filename=package://visualization/urdf/left_hand_v1_meshes/thumb_dist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
- added link left_thumb_metacarpol_link, mass 0.00864256984122037; collision mesh filename=package://visualization/urdf/left_hand_v1_meshes/thumb_meta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; visual mesh filename=package://visualization/urdf/left_hand_v1_meshes/thumb_meta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
- added link left_thumb_proximal_link, mass 0.0046151063369737; collision mesh filename=package://visualization/urdf/left_hand_v1_meshes/thumb_prox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; visual mesh filename=package://visualization/urdf/left_hand_v1_meshes/thumb_prox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
- added link left_thumb_tip_link, mass 0.00296168286968343; collision mesh filename=package://visualization/urdf/left_hand_v1_meshes/thumb_tip_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; visual mesh filename=package://visualization/urdf/left_hand_v1_meshes/thumb_tip_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
Joints:
- removed joint joint1
- removed joint joint2
- removed joint joint3
- removed joint joint4
- removed joint joint5
- removed joint joint6
- removed joint joint6_to_gripper_base
- removed joint joint7
- removed joint joint8
- added joint left_frame: type fixed, parent left_base_link, child left_frame_link, origin xyz=0 0 0 rpy=0 0 0, axis 0 0 0
- added joint left_index_dip: type revolute, parent left_index_middle_link, child left_index_distal_link, origin xyz=0 0.000383952941619931 0.0219966492934402 rpy=-0.00275677194064253 0 0, axis 1 0 0, limit lower=0 upper=1.5708 effort=0 velocity=0
- added joint left_index_mcp_abd: type revolute, parent left_frame_link, child left_index_f_link, origin xyz=-0.029596 -0.003707 0.1018 rpy=0 0 0.034907, axis 0 1 0, limit lower=-0.2618 upper=0.2618 effort=0 velocity=0
- added joint left_index_mcp_flex: type revolute, parent left_index_f_link, child left_index_proximal_link, origin xyz=0 -0.0004 0.0027 rpy=0.018103 0 0, axis 1 0 0, limit lower=0 upper=1.5708 effort=0 velocity=0
- added joint left_index_pip: type revolute, parent left_index_proximal_link, child left_index_middle_link, origin xyz=0 -0.000704692474492747 0.0430188505587838 rpy=0 0 0, axis 1 0 0, limit lower=0 upper=1.5708 effort=0 velocity=0
- added joint left_index_prismatic1: type prismatic, parent left_frame_link, child left_index_prismatic1_link, origin xyz=-0.0344747428096294 -0.00726357886481495 0.0945992626510313 rpy=0 0 0.0349065850398965, axis 0 0 -1, limit lower=0 upper=0.017 effort=0 velocity=0
- added joint left_index_prismatic2: type prismatic, parent left_frame_link, child left_index_prismatic2_link, origin xyz=-0.0244808345394687 -0.00691458389779098 0.0945992626518286 rpy=0 0 0.0349065850398965, axis 0 0 -1, limit lower=0 upper=0.017 effort=0 velocity=0
- added joint left_index_tip: type fixed, parent left_index_distal_link, child left_index_tip_link, origin xyz=0 0.00329764978643327 0.0249542326219998 rpy=0 0 0, axis 0 0 0
- added joint left_middle_dip: type revolute, parent left_middle_middle_link, child left_middle_distal_link, origin xyz=0 0.000383952941619943 0.0219966492934408 rpy=0 0 0, axis 1 0 0, limit lower=0 upper=1.5708 effort=0 velocity=0
- added joint left_middle_mcp_abd: type revolute, parent left_frame_link, child left_middle_f_link, origin xyz=-0.00849999999978476 -0.0026 0.1023 rpy=0 0 0, axis 0 1 0, limit lower=-0.2618 upper=0.2618 effort=0 velocity=0
- added joint left_middle_mcp_flex: type revolute, parent left_middle_f_link, child left_middle_proximal_link, origin xyz=0 -0.0004 0.0027 rpy=0.018103 0 0, axis 1 0 0, limit lower=0 upper=1.5708 effort=0 velocity=0
- added joint left_middle_pip: type revolute, parent left_middle_proximal_link, child left_middle_middle_link, origin xyz=0 -0.000704692474492743 0.0430188505587839 rpy=0 0 0, axis 1 0 0, limit lower=0 upper=1.5708 effort=0 velocity=0
- added joint left_middle_prismatic1: type prismatic, parent left_frame_link, child left_middle_prismatic1_link, origin xyz=-0.0134999999999849 -0.00598409580514471 0.0950947129912662 rpy=0 0 0, axis 0 0 -1, limit lower=0 upper=0.017 effort=0 velocity=0
- added joint left_middle_prismatic2: type prismatic, parent left_frame_link, child left_middle_prismatic2_link, origin xyz=-0.00350000000001516 -0.00598409580514471 0.0950947129920634 rpy=0 0 0, axis 0 0 -1, limit lower=0 upper=0.017 effort=0 velocity=0
- added joint left_middle_tip: type fixed, parent left_middle_distal_link, child left_middle_tip_link, origin xyz=0 0.00336643029687281 0.0249450469416905 rpy=-0.00275677194064254 0 0, axis 0 0 0
- added joint left_pinky_dip: type revolute, parent left_pinky_middle_link, child left_pinky_distal_link, origin xyz=0 0.000383952941619935 -0.0219966492934401 rpy=3.13883588164915 0 3.14159265358979, axis 1 0 0, limit lower=0 upper=1.5708 effort=0 velocity=0
- added joint left_pinky_mcp_abd: type revolute, parent left_frame_link, child left_pinky_f_link, origin xyz=0.0332259975438891 -0.00595751087982225 0.0890434920430963 rpy=0 0 -0.0699464803322307, axis 0 1 0, limit lower=-0.2618 upper=0.2618 effort=0 velocity=0
- added joint left_pinky_mcp_flex: type revolute, parent left_pinky_f_link, child left_pinky_proximal_link, origin xyz=0 -0.0004 0.0027 rpy=0.018103 0 0, axis 1 0 0, limit lower=0 upper=1.5708 effort=0 velocity=0
- added joint left_pinky_pip: type revolute, parent left_pinky_proximal_link, child left_pinky_middle_link, origin xyz=0 -0.000704692474492746 0.0430188505587839 rpy=3.14159265358978 0 3.14159265358979, axis -1 0 0, limit lower=0 upper=1.5708 effort=0 velocity=0
- added joint left_pinky_prismatic1: type prismatic, parent left_frame_link, child left_pinky_prismatic1_link, origin xyz=0.0280017112093865 -0.00898388440491384 0.0818382050343625 rpy=0 0 -0.0699464803322178, axis 0 0 -1, limit lower=0 upper=0.017 effort=0 velocity=0
- added joint left_pinky_prismatic2: type prismatic, parent left_frame_link, child left_pinky_prismatic2_link, origin xyz=0.0379772586307819 -0.00968277899130439 0.0818382050351598 rpy=0 0 -0.0699464803322178, axis 0 0 -1, limit lower=0 upper=0.017 effort=0 velocity=0
- added joint left_pinky_tip: type fixed, parent left_pinky_distal_link, child left_pinky_tip_link, origin xyz=0 0.00329764978643327 0.024954232622 rpy=0 0 0, axis 0 0 0
- added joint left_ring_dip: type revolute, parent left_ring_middle_link, child left_ring_distal_link, origin xyz=0 0.000383952941619927 0.0219966492934402 rpy=0 0 0, axis 1 0 0, limit lower=0 upper=1.5708 effort=0 velocity=0
- added joint left_ring_mcp_abd: type revolute, parent left_frame_link, child left_ring_f_link, origin xyz=0.0125958919149416 -0.00370704707588761 0.101804549659765 rpy=0 0 -0.0349065850398961, axis 0 1 0, limit lower=-0.2618 upper=0.2618 effort=0 velocity=0
- added joint left_ring_mcp_flex: type revolute, parent left_ring_f_link, child left_ring_proximal_link, origin xyz=0 -0.0004 0.0027 rpy=0.018103 0 0, axis 1 0 0, limit lower=0 upper=1.5708 effort=0 velocity=0
- added joint left_ring_pip: type revolute, parent left_ring_proximal_link, child left_ring_middle_link, origin xyz=0 -0.000704692474492746 0.0430188505587838 rpy=0 0 0, axis 1 0 0, limit lower=0 upper=1.5708 effort=0 velocity=0
- added joint left_ring_prismatic1: type prismatic, parent left_frame_link, child left_ring_prismatic1_link, origin xyz=0.00748083453946868 -0.00691458389779104 0.0945992626510313 rpy=0 0 -0.0349065850398832, axis 0 0 -1, limit lower=0 upper=0.017 effort=0 velocity=0
- added joint left_ring_prismatic2: type prismatic, parent left_frame_link, child left_ring_prismatic2_link, origin xyz=0.0174747428096295 -0.00726357886481505 0.0945992626518286 rpy=0 0 -0.0349065850398832, axis 0 0 -1, limit lower=0 upper=0.017 effort=0 velocity=0
- added joint left_ring_tip: type fixed, parent left_ring_distal_link, child left_ring_tip_link, origin xyz=0 0.00336643029687281 0.0249450469416905 rpy=-0.00275677194064252 0 0, axis 0 0 0
- added joint left_thumb_cmc_abd: type revolute, parent left_frame_link, child left_t_Link, origin xyz=-0.030369 -0.017851 0.02455 rpy=-1.2157 0.011469 1.5547, axis 0 -1 0, limit lower=0 upper=1.7453 effort=0 velocity=0
- added joint left_thumb_cmc_flex: type revolute, parent left_t_Link, child left_thumb_metacarpol_link, origin xyz=-0.00075443 -0.0051626 0.019636 rpy=0.14637 0.11355 -0.25937, axis 1 0 0, limit lower=0 upper=1.4000 effort=0 velocity=0
- added joint left_thumb_ip: type revolute, parent left_thumb_proximal_link, child left_thumb_distal_link, origin xyz=0 -0.009767 0.028366 rpy=0.34907 0 0, axis 1 0 0, limit lower=0 upper=1.5708 effort=0 velocity=0
- added joint left_thumb_mcp: type revolute, parent left_thumb_metacarpol_link, child left_thumb_proximal_link, origin xyz=0 0.0095039 0.034725 rpy=0 0 0, axis 1 0 0, limit lower=0 upper=1.2217 effort=0 velocity=0
- added joint left_thumb_tip: type fixed, parent left_thumb_distal_link, child left_thumb_tip_link, origin xyz=0 0.0023115858897875 0.029876683808909 rpy=0 0 0, axis 0 0 0
